File: hardware/kicad-v3/abb-welcome-gateway-v3.kicad_pcb (KiCad board)
At the start: 2 copper layers, 45.3 x 56.3 mm, 69 parts, among them P1 WJ500V-5.08-2P, Q1 S8050, Q2 S8050, Q3 S8050, Q4 2N7002, Q5 2N7002, Q6 2N7002, SW1 TS-1187A-B-A-B, U1 TPS5430DDAR, U2 ESP32-S3-WROOM-1-N16R8, U3 74LVC1G14

Commit message: fab: specify exact parts for P2 (1x6 2.54mm header) and U3 (SN74LVC1G14DBVR)
Both carried generic placeholders from the tscircuit conversion. Set the
manufacturer part in the symbol Value + footprint identity in schematic and
PCB, and refresh the BOM/pos exports. Metadata only; no copper change, DRC
still 0 errors / 0 unconnected. Documented in docs/STATUS.md.
Parts:
- P2: value (none) -> 61300611121; footprint tscircuit:chip -> tscircuit:PinHeader_1x06_2.54mm
- U3: value 74LVC1G14 -> SN74LVC1G14DBVR; footprint tscircuit:74LVC1G14 -> tscircuit:SOT-23-5
Changed lines of the file:
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@@
 		(embedded_fonts no)
 	)
-	(footprint "tscircuit:chip"
+	(footprint "tscircuit:PinHeader_1x06_2.54mm"
 		(layer "F.Cu")
 		(at 112.282 88.629)
@@
 			)
 		)
-		(property "Value" ""
+		(property "Value" "61300611121"
 			(at 0 3 0)
 			(layer "F.Fab")
@@
 		(embedded_fonts no)
 	)
-	(footprint "tscircuit:74LVC1G14"
+	(footprint "tscircuit:SOT-23-5"
 		(layer "F.Cu")
 		(at 88 91.9 180)
@@
 			)
 		)
-		(property "Value" "74LVC1G14"
+		(property "Value" "SN74LVC1G14DBVR"
 			(at 0 3 180)
 			(layer "F.Fab")
